File: HW/standalone/audi_concert1_chorus1_volume_fix/audi_concert1_chorus1_volume_fix.kicad_pcb (KiCad board)
At the start: 2 copper layers, 32.8 x 26.2 mm, 38 parts, among them CON1 I2C_to_TDA, CON2 USB, CON3 SPI_TO_PANEL, CON4 JLINK, U1 68HC05_PLCC, U2 AP1117-33, U3 STM32F103C8Tx, Y1 Crystal_GND24, Y2 Crystal_GND24

Commit message: v2.0 files
Parts:
- added C8: 10u/16V, Capacitors_Tantalum_SMD.pretty:TantalC_SizeA_EIA-3216_HandSoldering, B.Cu at (165.7, 115.3)
- added R20: 1k, Resistors_SMD.pretty:R_0805_HandSoldering, F.Cu at (180.1, 96.7)
- CON4: footprint Pin_Headers.pretty:Pin_Header_Straight_1x04 -> Pin_Headers.pretty:Pin_Header_Straight_1x06
- moved D1 12.0 mm to (185.9, 116.8)
- moved CON4 7.63 mm to (194.5, 95.6), turned to 0 degrees
- moved JP1 2.48 mm to (177.6, 97.6)
- moved C7 2.32 mm to (175.1, 96.6)
- moved C2 2.26 mm to (173.0, 96.6)
- moved R2 2.22 mm to (183.5, 115.8), turned to 270 degrees
- moved Y1 2.05 mm to (170.7, 97.0)
- moved JP2 1.82 mm to (178.8, 116.2)
- moved C3 1.77 mm to (168.5, 96.7)
- moved R3 1.58 mm to (181.4, 115.8)
- moved C1 0.56 mm to (176.3, 115.1)
- moved R1 0.36 mm to (173.9, 116.0)
- moved R13 0.15 mm to (190.1, 111.9)
- turned R14 to 180 degrees
Connections:
- CON4 pad 1: 3V3 -> GND
- CON4 pad 2: /SWDIO -> /SWDCLK
- CON4 pad 3: /SWDCLK -> /SWDIO
- CON4 pad 4: GND -> 3V3
- U1 pad 1: Net-(U1-Pad1) -> (no net)
- U1 pad 11: Net-(U1-Pad11) -> (no net)
- U1 pad 12: Net-(U1-Pad12) -> (no net)
- U1 pad 13: Net-(U1-Pad13) -> (no net)
- U1 pad 14: Net-(U1-Pad14) -> (no net)
- U1 pad 15: Net-(U1-Pad15) -> (no net)
- U1 pad 16: Net-(U1-Pad16) -> (no net)
- U1 pad 17: Net-(U1-Pad17) -> (no net)
- U1 pad 18: Net-(U1-Pad18) -> (no net)
- U1 pad 19: Net-(U1-Pad19) -> (no net)
- U1 pad 2: Net-(U1-Pad2) -> (no net)
- U1 pad 20: Net-(U1-Pad20) -> (no net)
- U1 pad 21: Net-(U1-Pad21) -> (no net)
- U1 pad 22: Net-(U1-Pad22) -> (no net)
- U1 pad 23: Net-(U1-Pad23) -> (no net)
- U1 pad 26: Net-(U1-Pad26) -> (no net)
- U1 pad 27: Net-(U1-Pad27) -> (no net)
- U1 pad 28: Net-(U1-Pad28) -> (no net)
- U1 pad 3: Net-(U1-Pad3) -> (no net)
- U1 pad 32: Net-(U1-Pad32) -> (no net)
- U1 pad 34: Net-(U1-Pad34) -> (no net)
- U1 pad 35: Net-(U1-Pad35) -> (no net)
- U1 pad 36: Net-(U1-Pad36) -> (no net)
- U1 pad 37: Net-(U1-Pad37) -> (no net)
- U1 pad 38: Net-(U1-Pad38) -> (no net)
- U1 pad 39: Net-(U1-Pad39) -> (no net)
- U1 pad 4: Net-(U1-Pad4) -> (no net)
- U1 pad 40: Net-(U1-Pad40) -> (no net)
- U1 pad 42: Net-(U1-Pad42) -> (no net)
- U1 pad 43: Net-(U1-Pad43) -> (no net)
- U1 pad 44: Net-(U1-Pad44) -> (no net)
- U1 pad 45: Net-(U1-Pad45) -> (no net)
- U1 pad 46: Net-(U1-Pad46) -> (no net)
- U1 pad 47: Net-(U1-Pad47) -> (no net)
- U1 pad 48: Net-(U1-Pad48) -> (no net)
- U1 pad 49: Net-(U1-Pad49) -> (no net)
- U1 pad 5: Net-(U1-Pad5) -> (no net)
- U1 pad 50: Net-(U1-Pad50) -> (no net)
- U1 pad 51: Net-(U1-Pad51) -> (no net)
- U1 pad 52: Net-(U1-Pad52) -> (no net)
- U1 pad 6: Net-(U1-Pad6) -> (no net)
- U1 pad 7: Net-(U1-Pad7) -> (no net)
- U1 pad 8: Net-(U1-Pad8) -> (no net)
- U1 pad 9: Net-(U1-Pad9) -> (no net)
- U3 pad 1: +BATT -> (no net)
- U3 pad 10: Net-(U3-Pad10) -> (no net)
- U3 pad 11: Net-(U3-Pad11) -> (no net)
- U3 pad 12: Net-(U3-Pad12) -> (no net)
- U3 pad 13: Net-(U3-Pad13) -> (no net)
- U3 pad 14: Net-(U3-Pad14) -> (no net)
- U3 pad 15: Net-(U3-Pad15) -> (no net)
- U3 pad 16: Net-(U3-Pad16) -> (no net)
- U3 pad 17: Net-(U3-Pad17) -> (no net)
- U3 pad 18: Net-(U3-Pad18) -> (no net)
- U3 pad 19: Net-(U3-Pad19) -> (no net)
- U3 pad 2: Net-(U3-Pad2) -> (no net)
- U3 pad 25: Net-(U3-Pad25) -> (no net)
- U3 pad 29: Net-(U3-Pad29) -> (no net)
- U3 pad 30: Net-(U3-Pad30) -> /TX
- U3 pad 31: Net-(U3-Pad31) -> /RX
- U3 pad 45: Net-(U3-Pad45) -> (no net)
- U3 pad 46: Net-(U3-Pad46) -> (no net)
Routing:
- net 3V3: track 75.9 -> 101.5 mm
- net /RX: track 0.00 -> 25.5 mm, vias 0 -> 1
- net /TX: track 0.00 -> 19.6 mm, vias 0 -> 1
- net Net-(D1-Pad1): track 20.1 -> 3.35 mm
- net /RESET: track 11.8 -> 21.3 mm, vias 0 -> 2
- net GND: track 105.2 -> 114.0 mm, vias 10 -> 14
- net /BOOT0: track 3.11 -> 8.40 mm
- net /RESET_KA: track 24.4 -> 29.2 mm
- net /SDA_TO_TDA: track 24.5 -> 28.1 mm
- net /SCL_TO_TDA: track 22.6 -> 25.7 mm, vias 2 -> 1
- net /DATA_FROM_MCU: track 4.69 -> 7.37 mm
- net /OSC32OUT: track 15.5 -> 18.1 mm
- net Net-(R19-Pad2): track 8.96 -> 10.7 mm
- net /USB+: track 9.37 -> 7.67 mm
- net Net-(CON2-Pad2): track 47.6 -> 46.0 mm
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Other:
- board text added: "AUDI"
- board text added: "chorus1"
- board text added: "concert1"
- board text added: "v2.0"
- board text added: "volume fix"
