File: HW/standalone/audi_concert1_chorus1_volume_fix/audi_concert1_chorus1_volume_fix.sch (KiCad schematic (older format))
At the start: 40 parts, among them CON1 I2C_to_TDA, CON2 USB, CON3 SPI_TO_PANEL, CON4 JLINK, SW1 SWITCH_DPST, U1 68HC05_PLCC, U2 AP1117-33, U3 STM32F103C8Tx, Y1 Crystal_GND24, Y2 Crystal_GND24

Commit message: v2.0 files
Parts:
- added R20: 1k, Resistors_SMD.pretty:R_0805_HandSoldering, symbol Device:R
- added R21: 2k2, Resistors_SMD.pretty:R_0805_HandSoldering, symbol Device:R
- added R22: 3k3, Resistors_SMD.pretty:R_0805_HandSoldering, symbol Device:R
- added U?: MAX809, TO_SOT_Packages_SMD.pretty:SOT-23, symbol MAX809_810:MAX809
- CON4: footprint Pin_Headers.pretty:Pin_Header_Straight_1x04 -> Pin_Headers.pretty:Pin_Header_Straight_1x06; symbol con:CONN_4 -> Connectors:CONN_1x6
Connections:
- net 3V3: now also CON4.4; no longer CON4.1
- net GND: now also CON4.1, R22.1, U?.1 (GND); no longer CON4.4
- net RESET: now also R20.2, R21.1, R22.2, U?.2 (RESET)
- net RESET_KA: now also R20.1
- net SWDCLK: now also CON4.2; no longer CON4.3
- net SWDIO: now also CON4.3; no longer CON4.2
- net RESET_MOTO: now reaches U1.18 (RESET)
- net RESET_MOTO: now also R21.2, U?.3 (VCC)
- net TX: now reaches U3.30 (TIM1_CH2/USART1_TX/PA9)
- net TX: now also CON4.6
- net RX: now reaches U3.31 (TIM1_CH3/USART1_RX/PA10)
- net RX: now also CON4.5
Other:
- note added: "3V when reset of moto goes to 5V"
- note added: "not populated"
- moved on the sheet: JP1, JP2
