File: HW/audi_concert1_chorus1_volume_fix/audi_concert1_chorus1_volume_fix.sch (KiCad schematic (older format))
At the start: 39 parts, among them CON1 I2C_to_TDA, CON2 USB, CON3 SPI_TO_PANEL, CON4 JLINK, U1 68HC05_PLCC, U2 AP1117-33, U3 STM32F103C8Tx, U4 MAX809, Y1 32.768kHz, Y2 8MHz

Commit message: v2.0
Signed-off-by: Tomas kovacik <nail@nodomain.sk>
Parts:
- added R1: 1k, Resistors_SMD.pretty:R_0805_HandSoldering, symbol Device:R
Connections:
- net GALA: now reaches U1.23 (TCAP2)
- net GALA: now also R1.1
- net at U3.10 (ADC1_IN0/ADC2_IN0/SYS_WKUP/TIM2_CH1/TIM2_ETR/USART2_CTS/PA0): now also R1.2
Changed lines of the file:
@@
-EESchema Schematic File Version 5
-LIBS:audi_concert1_chorus1_volume_fix-cache
-EELAYER 29 0
+EESchema Schematic File Version 4
+EELAYER 30 0
 EELAYER END
 $Descr A3 16535 11693
@@
 	1    0    0    -1
 $EndComp
+Wire Wire Line
+	5750 7550 5150 7550
+Text Label 5150 7550 0    50   ~ 0
+GALA
+Text Label 12200 3250 2    50   ~ 0
+GALA
+$Comp
+L Device:R R1
+U 1 1 5E7EA43A
+P 11750 3250
+F 0 "R1" V 11543 3250 50  0000 C CNN
+F 1 "1k" V 11634 3250 50  0000 C CNN
+F 2 "Resistors_SMD.pretty:R_0805_HandSoldering" V 11680 3250 50  0001 C CNN
+F 3 "~" H 11750 3250 50  0001 C CNN
+	1    11750 3250
+	0    1    1    0
+$EndComp
+Wire Wire Line
+	11600 3250 11250 3250
+Wire Wire Line
+	11900 3250 12200 3250
 $EndSCHEMATC
