File: HW/audi_concert1_chorus1_volume_fix/audi_concert1_chorus1_volume_fix.sch (KiCad schematic (older format))
At the start: 40 parts, among them CON1 I2C_to_TDA, CON2 USB, CON3 SPI_TO_PANEL, CON4 JLINK, U1 68HC05_PLCC, U2 AP1117-33, U3 STM32F103C8Tx, U4 MAX809, Y1 32.768kHz, Y2 8MHz

Commit message: HW v3
Parts:
- added R21, R22: 10k, Resistors_SMD.pretty:R_0805_HandSoldering, symbol Device:R
Connections:
- net DATA_FROM_MCU: now also R21.1
- net DATA_TO_PANEL: now also CON3.1, R22.1; no longer CON3.2
- net STATUS_TO_PANEL: now also CON3.2; no longer CON3.1
- net at R17.2: now also U3.25 (PB12/I2C2_SMBA/SPI2_NSS/TIM1_BKIN/USART3_CK); no longer U3.28 (PB15/ADC1_EXTI15/ADC2_EXTI15/SPI2_MOSI/TIM1_CH3N)
- net at U3.41 (PB5/I2C1_SMBA/SPI1_MOSI/TIM3_CH2): now also R21.2; no longer R19.2
- net at U3.45 (PB8/CAN_RX/I2C1_SCL/TIM4_CH3): now also R19.2
- new net: R22.2, U3.28 (PB15/ADC1_EXTI15/ADC2_EXTI15/SPI2_MOSI/TIM1_CH3N)
Other:
- moved on the sheet: R17, R19

Commit message: HW3
Signed-off-by: Tomas kovacik <nail@nodomain.sk>
Parts:
- added Q1, Q2: BSS138, TO_SOT_Packages_SMD:SOT-23, symbol Transistor_FET:BSS138
- added R23, R24: 10k, Resistors_SMD.pretty:R_0805_HandSoldering, symbol Device:R
Connections:
- net 3V3: now also R23.2, R24.2
- net GND: now also Q1.2 (S), Q2.2 (S)
- net at R11.1: now also Q2.1 (G); no longer U3.38 (ADC1_EXTI15/ADC2_EXTI15/SPI1_NSS/SYS_JTDI/TIM2_CH1/TIM2_ETR/PA15)
- net at R17.2: now also Q1.1 (G); no longer U3.25 (PB12/I2C2_SMBA/SPI2_NSS/TIM1_BKIN/USART3_CK)
- net at U3.14 (ADC1_IN4/ADC2_IN4/SPI1_NSS/USART2_CK/PA4): now also Q2.3 (D), R24.1
- new net: Q1.3 (D), R23.1, U3.25 (PB12/I2C2_SMBA/SPI2_NSS/TIM1_BKIN/USART3_CK)
Other:
- moved on the sheet: R17
Changed lines of the file:
@@
 Connection ~ 4870 4650
 Connection ~ 4850 3650
+Connection ~ 12270 3650
+Connection ~ 3630 4450
 Wire Wire Line
 	1500 850  2100 850
@@
 	2000 3950 1500 3950
 Wire Wire Line
+	2110 4980 2900 4980
+Wire Wire Line
 	2300 3950 2450 3950
 Wire Wire Line
@@
 	2450 3950 2850 3950
 Wire Wire Line
+	3200 4980 3330 4980
+Wire Wire Line
+	3630 3740 3630 3990
+Wire Wire Line
+	3630 4450 3630 4290
+Wire Wire Line
+	3630 4450 3630 4780
+Wire Wire Line
+	3630 4450 5450 4450
+Wire Wire Line
+	3630 5180 3630 5300
+Wire Wire Line
 	4150 3550 4900 3550
 Wire Wire Line
@@
 	4250 3950 4900 3950
 Wire Wire Line
-	4250 4450 4900 4450
-Wire Wire Line
 	4250 4550 4900 4550
 Wire Wire Line
@@
 	5200 4050 5450 4050
 Wire Wire Line
-	5200 4450 5450 4450
-Wire Wire Line
 	5200 4550 5450 4550
 Wire Wire Line
@@
 	9800 5550 10550 5550
 Wire Wire Line
-	10850 5550 11350 5550
+	10850 5550 11970 5550
+Wire Wire Line
+	11250 3650 12270 3650
 Wire Wire Line
 	11250 4150 11750 4150
@@
 	11250 4650 11750 4650
 Wire Wire Line
-	11250 4750 11350 4750
-Wire Wire Line
-	11350 5550 11350 4750
-Wire Wire Line
 	11600 3250 11250 3250
 Wire Wire Line
@@
 Wire Wire Line
 	12250 8700 11950 8700
+Wire Wire Line
+	12270 2330 12270 2580
+Wire Wire Line
+	12270 2880 12270 3650
+Wire Wire Line
+	12270 3650 12270 5350
+Wire Wire Line
+	12270 5750 12270 5870
 Wire Wire Line
 	12550 9000 12550 9300
@@
 Text Notes 2150 5250 2    50   ~ 0
 *
-Text Notes 4250 4500 2    50   ~ 0
+Text Notes 3860 4470 2    50   ~ 0
 *
 Text Label 1900 2650 2    50   ~ 0
@@
 Text Label 2100 1450 2    50   ~ 0
 SWDCLK
+Text Label 2110 4980 0    50   ~ 0
+STATUS_TO_PANEL
 Text Label 2150 5450 2    50   ~ 0
 CLOCK_TO_PANEL
@@
 Text Label 4250 4050 0    50   ~ 0
 RESET_KA
-Text Label 4250 4450 0    50   ~ 0
-STATUS_TO_PANEL
 Text Label 4250 4550 0    50   ~ 0
 CLOCK_TO_PANEL
@@
 $EndComp
 $Comp
+L audi_concert1_chorus1_volume_fix-rescue:3V3-pwr #PWR015
+U 1 1 5E9DF5EE
+P 3630 3740
+F 0 "#PWR015" H 3630 3700 30  0001 C CNN
+F 1 "3V3" H 3655 3901 60  0000 C CNN
+F 2 "" H 3630 3740 50  0001 C CNN
+F 3 "" H 3630 3740 50  0001 C CNN
+	1    3630 3740
+	1    0    0    -1
+$EndComp
+$Comp
 L audi_concert1_chorus1_volume_fix-rescue:5V-pwr #PWR0103
 U 1 1 5AD01E63
@@
 $EndComp
 $Comp
+L audi_concert1_chorus1_volume_fix-rescue:3V3-pwr #PWR017
+U 1 1 5E9DC3BF
+P 12270 2330
+F 0 "#PWR017" H 12270 2290 30  0001 C CNN
+F 1 "3V3" H 12295 2491 60  0000 C CNN
+F 2 "" H 12270 2330 50  0001 C CNN
+F 3 "" H 12270 2330 50  0001 C CNN
+	1    12270 2330
+	1    0    0    -1
+$EndComp
+$Comp
 L audi_concert1_chorus1_volume_fix-rescue:3V3-pwr #PWR09
 U 1 1 5AD4F28B
@@
 $EndComp
 $Comp
+L power:GND #PWR016
+U 1 1 5E9E46CA
+P 3630 5300
+F 0 "#PWR016" H 3630 5050 50  0001 C CNN
+F 1 "GND" H 3635 5127 50  0000 C CNN
+F 2 "" H 3630 5300 50  0001 C CNN
+F 3 "" H 3630 5300 50  0001 C CNN
+	1    3630 5300
+	1    0    0    -1
+$EndComp
+$Comp
 L power:GND #PWR0101
 U 1 1 5AD0005D
@@
 F 3 "" H 11950 9300 50  0001 C CNN
 	1    11950 9300
+	1    0    0    -1
+$EndComp
+$Comp
+L power:GND #PWR018
+U 1 1 5E9D6061
+P 12270 5870
+F 0 "#PWR018" H 12270 5620 50  0001 C CNN
+F 1 "GND" H 12275 5697 50  0000 C CNN
+F 2 "" H 12270 5870 50  0001 C CNN
+F 3 "" H 12270 5870 50  0001 C CNN
+	1    12270 5870
 	1    0    0    -1
 $EndComp
@@
 $EndComp
 $Comp
+L Device:R R17
+U 1 1 5AE4CD58
+P 3050 4980
+F 0 "R17" V 3050 4980 50  0000 C CNN
+F 1 "1k" V 3100 4830 50  0000 C CNN
+F 2 "Resistors_SMD.pretty:R_0805_HandSoldering" V 2980 4980 50  0001 C CNN
+F 3 "~" H 3050 4980 50  0001 C CNN
+	1    3050 4980
+	0    -1   1    0
+$EndComp
+$Comp
+L Device:R R23
+U 1 1 5E9DF5DF
+P 3630 4140
+F 0 "R23" V 3630 4140 50  0000 C CNN
+F 1 "10k" V 3580 3990 50  0000 C CNN
+F 2 "Resistors_SMD.pretty:R_0805_HandSoldering" V 3560 4140 50  0001 C CNN
+F 3 "~" H 3630 4140 50  0001 C CNN
+	1    3630 4140
+	-1   0    0    1
+$EndComp
+$Comp
 L Device:R R20
 U 1 1 5BE1DE4B
@@
 $EndComp
 $Comp
-L Device:R R17
-U 1 1 5AE4CD58
-P 5050 4450
-F 0 "R17" V 5050 4450 50  0000 C CNN
-F 1 "1k" V 5100 4300 50  0000 C CNN
-F 2 "Resistors_SMD.pretty:R_0805_HandSoldering" V 4980 4450 50  0001 C CNN
-F 3 "~" H 5050 4450 50  0001 C CNN
-	1    5050 4450
-	0    -1   1    0
-$EndComp
-$Comp
 L Device:R R15
 U 1 1 5AE4CC42
@@
 $EndComp
 $Comp
+L Device:R R24
+U 1 1 5E9D8E83
+P 12270 2730
+F 0 "R24" V 12270 2730 50  0000 C CNN
+F 1 "10k" V 12220 2580 50  0000 C CNN
+F 2 "Resistors_SMD.pretty:R_0805_HandSoldering" V 12200 2730 50  0001 C CNN
+F 3 "~" H 12270 2730 50  0001 C CNN
+	1    12270 2730
+	-1   0    0    1
+$EndComp
+$Comp
 L Device:R R18
 U 1 1 5AD78EBB
@@
 $EndComp
 $Comp
+L Transistor_FET:BSS138 Q1
+U 1 1 5E9E46B8
+P 3530 4980
+F 0 "Q1" H 3736 5025 50  0000 L CNN
+F 1 "BSS138" H 3736 4935 50  0000 L CNN
+F 2 "TO_SOT_Packages_SMD:SOT-23" H 3730 4905 50  0001 L CIN
+F 3 "https://www.fairchildsemi.com/datasheets/BS/BSS138.pdf" H 3530 4980 50  0001 L CNN
+	1    3530 4980
+	1    0    0    -1
+$EndComp
+$Comp
+L Transistor_FET:BSS138 Q2
+U 1 1 5E9D1DC2
+P 12170 5550
+F 0 "Q2" H 12376 5595 50  0000 L CNN
+F 1 "BSS138" H 12376 5505 50  0000 L CNN
+F 2 "TO_SOT_Packages_SMD:SOT-23" H 12370 5475 50  0001 L CIN
+F 3 "https://www.fairchildsemi.com/datasheets/BS/BSS138.pdf" H 12170 5550 50  0001 L CNN
+	1    12170 5550
+	1    0    0    -1
+$EndComp
+$Comp
