File: HW/audi_concert1_chorus1_volume_fix/audi_concert1_chorus1_volume_fix_v3.kicad_sch (KiCad schematic)
At the start: 46 parts, among them CON1 I2C_to_TDA, CON2 USB, CON3 SPI_TO_PANEL, CON4 JLINK, Q1 BSS138, Q2 BSS138, U1 68HC05_PLCC, U2 AP1117-33, U3 STM32F103C8Tx, U4 MAX809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

Commit message: HW v4
Parts:
- CON3: value SPI_TO_PANEL -> NP
- Q1, Q2: value BSS138 -> NP
- R15, R16, R17: value 1k -> NP
- R22, R23, R24: value 10k -> NP

Commit message: notes
Parts:
- added R25, R26: 0, Resistors_SMD.pretty:R_0603, symbol Device:R
- CON3: value NP -> SPI_TO_PANEL
- R15, R16, R17: value NP -> 1k
- R21: value 10k -> NP
Connections:
- net at Q2.1 (G), R11.1: now also R26.1
- net at Q1.1 (G), R17.2: now also R25.1
- net at Q2.3 (D), R24.1, U3.14 (ADC1_IN4/ADC2_IN4/SPI1_NSS/USART2_CK/PA4): now also R26.2
- net at Q1.3 (D), R23.1, U3.25 (PB12/I2C2_SMBA/SPI2_NSS/TIM1_BKIN/USART3_CK): now also R25.2
Other:
- note added: "FIX"
Changed lines of the file:
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@@
   )
   (junction (at 62.23 100.33))
+  (junction (at 82.9818 126.492))
   (junction (at 92.202 113.03))
+  (junction (at 92.202 119.126))
   (junction (at 123.19 92.71))
   (junction (at 123.698 118.11))
@@
   (junction (at 212.09 35.56))
   (junction (at 212.09 135.89))
+  (junction (at 298.577 140.97))
   (junction (at 303.53 220.98))
   (junction (at 311.658 92.71))
+  (junction (at 311.658 131.5212))
   (junction (at 332.74 110.49))
   (junction (at 332.74 220.98))
@@
     (stroke (width 0) (type solid) (color 0 0 0 0))
   )
-  (wire (pts (xy 81.28 126.492) (xy 84.582 126.492))
+  (wire (pts (xy 81.28 126.492) (xy 82.9818 126.492))
+    (stroke (width 0) (type solid) (color 0 0 0 0))
+  )
+  (wire (pts (xy 82.9818 119.126) (xy 82.9818 126.492))
+    (stroke (width 0) (type solid) (color 0 0 0 0))
+  )
+  (wire (pts (xy 82.9818 126.492) (xy 84.582 126.492))
+    (stroke (width 0) (type solid) (color 0 0 0 0))
+  )
+  (wire (pts (xy 83.439 119.126) (xy 82.9818 119.126))
     (stroke (width 0) (type solid) (color 0 0 0 0))
   )
@@
     (stroke (width 0) (type solid) (color 0 0 0 0))
   )
-  (wire (pts (xy 92.202 113.03) (xy 92.202 121.412))
+  (wire (pts (xy 92.202 113.03) (xy 92.202 119.126))
     (stroke (width 0) (type solid) (color 0 0 0 0))
   )
@@
     (stroke (width 0) (type solid) (color 0 0 0 0))
   )
+  (wire (pts (xy 92.202 119.126) (xy 91.059 119.126))
+    (stroke (width 0) (type solid) (color 0 0 0 0))
+  )
+  (wire (pts (xy 92.202 119.126) (xy 92.202 121.412))
+    (stroke (width 0) (type solid) (color 0 0 0 0))
+  )
   (wire (pts (xy 92.202 131.572) (xy 92.202 134.62))
     (stroke (width 0) (type solid) (color 0 0 0 0))
@@
     (stroke (width 0) (type solid) (color 0 0 0 0))
   )
-  (wire (pts (xy 275.59 140.97) (xy 304.038 140.97))
+  (wire (pts (xy 275.59 140.97) (xy 298.577 140.97))
     (stroke (width 0) (type solid) (color 0 0 0 0))
   )
@@
     (stroke (width 0) (type solid) (color 0 0 0 0))
   )
+  (wire (pts (xy 298.577 131.5212) (xy 298.577 140.97))
+    (stroke (width 0) (type solid) (color 0 0 0 0))
+  )
+  (wire (pts (xy 298.577 140.97) (xy 304.038 140.97))
+    (stroke (width 0) (type solid) (color 0 0 0 0))
+  )
+  (wire (pts (xy 300.7106 131.5212) (xy 298.577 131.5212))
+    (stroke (width 0) (type solid) (color 0 0 0 0))
+  )
   (wire (pts (xy 302.26 82.55) (xy 309.88 82.55))
     (stroke (width 0) (type solid) (color 0 0 0 0))
@@
     (stroke (width 0) (type solid) (color 0 0 0 0))
   )
-  (wire (pts (xy 311.658 92.71) (xy 311.658 135.89))
+  (wire (pts (xy 311.658 92.71) (xy 311.658 131.5212))
+    (stroke (width 0) (type solid) (color 0 0 0 0))
+  )
+  (wire (pts (xy 311.658 131.5212) (xy 308.3306 131.5212))
+    (stroke (width 0) (type solid) (color 0 0 0 0))
+  )
+  (wire (pts (xy 311.658 131.5212) (xy 311.658 135.89))
     (stroke (width 0) (type solid) (color 0 0 0 0))
   )
@@
     (effects (font (size 1.27 1.27)) (justify right bottom))
   )
+  (text "FIX" (at 83.6676 118.5672 180)
+    (effects (font (size 1.27 1.27)) (justify right bottom))
+  )
   (text "*" (at 98.044 113.538 180)
+    (effects (font (size 1.27 1.27)) (justify right bottom))
+  )
+  (text "FIX" (at 300.6598 131.3942 180)
     (effects (font (size 1.27 1.27)) (justify right bottom))
   )
@@
     (in_bom yes)
     (property "Reference" "R17" (id 0) (at 77.47 126.492 90))
-    (property "Value" "NP" (id 1) (at 81.28 127.762 90))
+    (property "Value" "1k" (id 1) (at 81.28 127.762 90))
     (property "Footprint" "Resistors_SMD.pretty:R_0805_HandSoldering" (id 2) (at 77.47 124.714 90)
       (effects (font (size 1.27 1.27)) hide)
     )
     (property "Datasheet" "~" (id 3) (at 77.47 126.492 0)
+      (effects (font (size 1.27 1.27)) hide)
+    )
+  )
+  (symbol (lib_id "Device:R") (at 87.249 119.126 90) (mirror x) (unit 1)
+    (in_bom yes)
+    (property "Reference" "R25" (id 0) (at 87.249 119.126 90))
+    (property "Value" "0" (id 1) (at 91.0588 120.3956 90))
+    (property "Footprint" "Resistors_SMD.pretty:R_0603" (id 2) (at 87.249 117.348 90)
+      (effects (font (size 1.27 1.27)) hide)
+    )
+    (property "Datasheet" "~" (id 3) (at 87.249 119.126 0)
       (effects (font (size 1.27 1.27)) hide)
     )
@@
     (in_bom yes)
     (property "Reference" "R21" (id 0) (at 128.27 95.25 90))
-    (property "Value" "10k" (id 1) (at 132.08 96.52 90))
+    (property "Value" "NP" (id 1) (at 132.08 96.52 90))
     (property "Footprint" "Resistors_SMD.pretty:R_0805_HandSoldering" (id 2) (at 128.27 97.028 90)
       (effects (font (size 1.27 1.27)) hide)
@@
     (in_bom yes)
     (property "Reference" "R15" (id 0) (at 128.27 115.57 90))
-    (property "Value" "NP" (id 1) (at 132.08 116.84 90))
+    (property "Value" "1k" (id 1) (at 132.08 116.84 90))
     (property "Footprint" "Resistors_SMD.pretty:R_0805_HandSoldering" (id 2) (at 128.27 113.792 90)
       (effects (font (size 1.27 1.27)) hide)
@@
     (in_bom yes)
     (property "Reference" "R16" (id 0) (at 128.27 118.11 90))
-    (property "Value" "NP" (id 1) (at 132.08 119.38 90))
+    (property "Value" "1k" (id 1) (at 132.08 119.38 90))
     (property "Footprint" "Resistors_SMD.pretty:R_0805_HandSoldering" (id 2) (at 128.27 116.332 90)
       (effects (font (size 1.27 1.27)) hide)
@@
     )
   )
+  (symbol (lib_id "Device:R") (at 304.5206 131.5212 90) (mirror x) (unit 1)
+    (in_bom yes)
+    (property "Reference" "R26" (id 0) (at 304.5206 131.5212 90))
+    (property "Value" "0" (id 1) (at 308.3304 132.7908 90))
+    (property "Footprint" "Resistors_SMD.pretty:R_0603" (id 2) (at 304.5206 129.7432 90)
+      (effects (font (size 1.27 1.27)) hide)
+    )
+    (property "Datasheet" "~" (id 3) (at 304.5206 131.5212 0)
+      (effects (font (size 1.27 1.27)) hide)
+    )
+  )
   (symbol (lib_id "Device:R") (at 311.658 69.342 180) (unit 1)
     (in_bom yes)
@@
       (effects (font (size 1.524 1.524)))
     )
-    (property "Value" "NP" (id 1) (at 32.537 134.849 0)
+    (property "Value" "SPI_TO_PANEL" (id 1) (at 32.5374 134.8486 0)
       (effects (font (size 1.524 1.524)))
     )
@@
       (reference "R24") (unit 1)
     )
+    (path "/e820c174-aed1-4aa2-a5cc-bacc3a6f8c65"
+      (reference "R25") (unit 1)
+    )
+    (path "/f519c534-a4e0-4f4e-93a2-ee27eeaaf2c1"
+      (reference "R26") (unit 1)
+    )
     (path "/00000000-0000-0000-0000-00005acfff11"

Commit message: fix resistors are 0805
Parts:
- R25, R26: footprint Resistors_SMD.pretty:R_0603 -> Resistors_SMD.pretty:R_0805
Changed lines of the file:
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@@
     (property "Reference" "R25" (id 0) (at 87.249 119.126 90))
     (property "Value" "0" (id 1) (at 91.0588 120.3956 90))
-    (property "Footprint" "Resistors_SMD.pretty:R_0603" (id 2) (at 87.249 117.348 90)
+    (property "Footprint" "Resistors_SMD.pretty:R_0805" (id 2) (at 87.249 117.348 90)
       (effects (font (size 1.27 1.27)) hide)
     )
@@
     (property "Reference" "R26" (id 0) (at 304.5206 131.5212 90))
     (property "Value" "0" (id 1) (at 308.3304 132.7908 90))
-    (property "Footprint" "Resistors_SMD.pretty:R_0603" (id 2) (at 304.5206 129.7432 90)
-      (effects (font (size 1.27 1.27)) hide)
-    )
+    (property "Footprint" "Resistors_SMD.pretty:R_0805" (id 2) (at 304.5206 129.7432 90)
+      (effects (font (size 1.27 1.27)) hide)
+    )
