File: HW/audi_concert1_chorus1_volume_fix/audi_concert1_chorus1_volume_fix_v3.kicad_pcb (KiCad board)
At the start: 2 copper layers, 34 x 26.2 mm, 46 parts, among them CON1 I2C_to_TDA, CON2 USB, CON3 SPI_TO_PANEL, CON4 JLINK, Q1 BSS138, Q2 BSS138, U1 68HC05_PLCC, U2 AP1117-33, U3 STM32F103C8Tx, U4 MAX809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

Commit message: HW v4
Parts:
- CON3: value SPI_TO_PANEL -> NP
- R7: footprint Resistors_SMD.pretty:R_0603_HandSoldering -> Resistors_SMD.pretty:R_0805_HandSoldering
- _: renamed from R22; value 10k -> NP
- _: renamed from Q1; value BSS138 -> NP
- _: renamed from R16; value 1k -> NP
- _: renamed from R15; value 1k -> NP
- _: renamed from R17; value 1k -> NP
- _: renamed from R23; value 10k -> NP
- _: renamed from R24; value 10k -> NP
- _: renamed from Q2; value BSS138 -> NP
Other:
- board text added: "wirebridge"
- board text removed: "CLK DATA"
- board text removed: "CL|DA|ST"
- board text removed: "STA TUS"

Commit message: fix for v3 HW
Parts:
- added R25: 0, Resistors_SMD.pretty:R_0805, F.Cu at (127.4, 93.9)
- added R26: 0, Resistors_SMD.pretty:R_0805, F.Cu at (127.5, 80.4)
- CON3: value NP -> SPI_TO_PANEL
- R15, R16, R17: renamed from _; value NP -> 1k
- R21: value 10k -> NP
- renumbered _ to Q1, _ to Q2, _ to R22, _ to R23, _ to R24
Other:
- board text removed: "wirebridge"
Changed lines of the file:
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@@
   (general
     (thickness 1.6)
-    (drawings 22)
+    (drawings 19)
     (tracks 756)
-    (modules 46)
+    (modules 48)
     (nets 48)
   )
@@
     (uvia_drill 0.1)
   )
+  (module "Resistors_SMD.pretty:R_0805" (layer "F.Cu")
+    (at 127.479992 80.411487 155)
+    (descr "Resistor SMD 0805, reflow soldering, Vishay (see dcrcw.pdf)")
+    (tags "resistor 0805")
+    (attr smd)
+    (fp_text reference "R26" (at 2.51131 0.042658 245) (layer "F.SilkS")
+      (effects (font (size 1 1) (thickness 0.15)))
+    )
+    (fp_text value "0" (at 0 2.1 155) (layer "F.Fab")
+      (effects (font (size 1 1) (thickness 0.15)))
+    )
+    (fp_line (start -0.6 -0.875) (end 0.6 -0.875) (layer "F.SilkS") (width 0.15))
+    (fp_line (start 0.6 0.875) (end -0.6 0.875) (layer "F.SilkS") (width 0.15))
+    (fp_line (start 1.6 -1) (end 1.6 1) (layer "F.CrtYd") (width 0.05))
+    (fp_line (start -1.6 -1) (end -1.6 1) (layer "F.CrtYd") (width 0.05))
+    (fp_line (start -1.6 1) (end 1.6 1) (layer "F.CrtYd") (width 0.05))
+    (fp_line (start -1.6 -1) (end 1.6 -1) (layer "F.CrtYd") (width 0.05))
+    (pad "2" smd rect (at 0.95 0 155) (size 0.7 1.3) (layers "F.Cu" "F.Paste" "F.Mask")
+      (net 47 "Net-(Q2-Pad3)"))
+    (pad "1" smd rect (at -0.95 0 155) (size 0.7 1.3) (layers "F.Cu" "F.Paste" "F.Mask")
+      (net 44 "Net-(Q2-Pad1)"))
+    (model "Resistors_SMD.3dshapes/R_0805.wrl"
+      (at (xyz 0 0 0))
+      (scale (xyz 1 1 1))
+      (rotate (xyz 0 0 0))
+    )
+  )
+  (module "Resistors_SMD.pretty:R_0805" (layer "F.Cu")
+    (at 127.381 93.853 -25)
+    (descr "Resistor SMD 0805, reflow soldering, Vishay (see dcrcw.pdf)")
+    (tags "resistor 0805")
+    (attr smd)
+    (fp_text reference "R25" (at 2.604667 0.326843 245) (layer "F.SilkS")
+      (effects (font (size 1 1) (thickness 0.15)))
+    )
+    (fp_text value "0" (at 0 2.1 155) (layer "F.Fab")
+      (effects (font (size 1 1) (thickness 0.15)))
+    )
+    (fp_line (start -0.6 -0.875) (end 0.6 -0.875) (layer "F.SilkS") (width 0.15))
+    (fp_line (start 0.6 0.875) (end -0.6 0.875) (layer "F.SilkS") (width 0.15))
+    (fp_line (start 1.6 -1) (end 1.6 1) (layer "F.CrtYd") (width 0.05))
+    (fp_line (start -1.6 -1) (end -1.6 1) (layer "F.CrtYd") (width 0.05))
+    (fp_line (start -1.6 1) (end 1.6 1) (layer "F.CrtYd") (width 0.05))
+    (fp_line (start -1.6 -1) (end 1.6 -1) (layer "F.CrtYd") (width 0.05))
+    (pad "2" smd rect (at 0.95 0 335) (size 0.7 1.3) (layers "F.Cu" "F.Paste" "F.Mask")
+      (net 46 "Net-(Q1-Pad3)"))
+    (pad "1" smd rect (at -0.95 0 335) (size 0.7 1.3) (layers "F.Cu" "F.Paste" "F.Mask")
+      (net 45 "Net-(Q1-Pad1)"))
+    (model "Resistors_SMD.3dshapes/R_0805.wrl"
+      (at (xyz 0 0 0))
+      (scale (xyz 1 1 1))
+      (rotate (xyz 0 0 0))
+    )
+  )
   (module "Resistors_SMD.pretty:R_0805_HandSoldering" (layer "F.Cu")
     (at 124.6124 73.9902 -90)
@@
     (tags "resistor 0805")
     (attr smd)
-    (fp_text reference "_" (at -0.0127 -0.0635 90) (layer "F.SilkS")
+    (fp_text reference "R22" (at -0.0127 -0.0635 90) (layer "F.SilkS")
       (effects (font (size 0.6 0.6) (thickness 0.1)))
     )
@@
     (tags "SOT-23")
     (attr smd)
-    (fp_text reference "_" (at 0.6858 1.84404) (layer "F.SilkS")
+    (fp_text reference "Q1" (at 0.6858 1.84404) (layer "F.SilkS") hide
       (effects (font (size 1 1) (thickness 0.15)))
     )
@@
     (tags "resistor 0805")
     (attr smd)
-    (fp_text reference "_" (at -0.0508 -0.0254) (layer "F.SilkS")
+    (fp_text reference "R16" (at -0.0508 -0.0254) (layer "F.SilkS")
       (effects (font (size 0.6 0.6) (thickness 0.1)))
     )
-    (fp_text value "NP" (at -0.00254 0.09652 90) (layer "F.Fab")
+    (fp_text value "1k" (at -0.00254 0.09652 90) (layer "F.Fab")
       (effects (font (size 1 1) (thickness 0.15)))
     )
@@
     (tags "resistor 0805")
     (attr smd)
-    (fp_text reference "_" (at 0 0 180) (layer "F.SilkS")
+    (fp_text reference "R15" (at 0 0 180) (layer "F.SilkS")
       (effects (font (size 0.6 0.6) (thickness 0.1)))
     )
-    (fp_text value "NP" (at 0.03556 -0.07874 270) (layer "F.Fab")
+    (fp_text value "1k" (at 0.03556 -0.07874 270) (layer "F.Fab")
       (effects (font (size 1 1) (thickness 0.15)))
     )
@@
     (tags "resistor 0805")
     (attr smd)
-    (fp_text reference "_" (at -0.0216 -0.0254) (layer "B.SilkS")
+    (fp_text reference "R17" (at -0.0216 -0.0254) (layer "B.SilkS")
       (effects (font (size 0.6 0.6) (thickness 0.1)) (justify mirror))
     )
-    (fp_text value "NP" (at -0.12828 -0.04826 -90) (layer "B.Fab")
+    (fp_text value "1k" (at -0.12828 -0.04826 -90) (layer "B.Fab")
       (effects (font (size 1 1) (thickness 0.15)) (justify mirror))
     )
@@
       (effects (font (size 0.8 0.8) (thickness 0.1)))
     )
-    (fp_text value "10k" (at 0.1778 0.0254 90) (layer "F.Fab")
+    (fp_text value "NP" (at 0.1778 0.0254 90) (layer "F.Fab")
       (effects (font (size 1 1) (thickness 0.15)))
     )
@@
     (tags "resistor 0805")
     (attr smd)
-    (fp_text reference "_" (at -0.04826 -0.09398 180) (layer "F.SilkS")
+    (fp_text reference "R23" (at -0.04826 -0.09398 180) (layer "F.SilkS")
       (effects (font (size 0.6 0.6) (thickness 0.1)))
     )
@@
     (tags "resistor 0805")
     (attr smd)
-    (fp_text reference "_" (at 0.0635 -0.1163 180) (layer "B.SilkS")
+    (fp_text reference "R24" (at 0.0635 -0.1163 180) (layer "B.SilkS")
       (effects (font (size 0.6 0.6) (thickness 0.1)) (justify mirror))
     )
@@
     (tags "SOT-23")
     (attr smd)
-    (fp_text reference "_" (at 1.68656 -1.45796) (layer "F.SilkS")
+    (fp_text reference "Q2" (at 1.68656 -1.45796) (layer "F.SilkS") hide
       (effects (font (size 1 1) (thickness 0.15)))
     )
@@
       (effects (font (size 0.6 0.6) (thickness 0.1)))
     )
-    (fp_text value "NP" (at 3.07594 4.318 180) (layer "F.Fab")
+    (fp_text value "SPI_TO_PANEL" (at 3.07594 4.318 180) (layer "F.Fab")
       (effects (font (size 1 1) (thickness 0.15)))
     )
@@
     )
   )
-  (gr_line (start 128.5875 80.5307) (end 143.9545 80.5307) (layer "F.SilkS") (width 0.12))
-  (gr_text "wirebridge" (at 140.3477 79.8703) (layer "F.SilkS")
-    (effects (font (size 1 1) (thickness 0.15)))
-  )
-  (gr_line (start 126.492 79.9465) (end 128.4986 80.9879) (layer "F.SilkS") (width 1))
   (gr_text "5V" (at 103.0986 89.3572) (layer "F.SilkS")
     (effects (font (size 1 1) (thickness 0.15)))
