File: HW/audi_concert1_chorus1_volume_fix/audi_concert1_chorus1_volume_fix.kicad_sch (KiCad schematic)
At the start: 42 parts, among them CON1 I2C_to_TDA, CON2 USB, CON3 SPI_TO_PANEL, CON4 JLINK, U1 68HC05_PLCC, U2 AP1117-33, U3 STM32F103C8Tx, U4 MAX809, Y1 32.768kHz, Y2 8MHz

Commit message: gala input fix 11+10 togeter
Connections:
- net at R4.1: now also U3.15 (ADC1_IN5/ADC2_IN5/SPI1_SCK/PA5); no longer U3.39 (PB3/SPI1_SCK/SYS_JTDO-TRACESWO/TIM2_CH2)
- net at R5.2: now also U3.16 (ADC1_IN6/ADC2_IN6/SPI1_MISO/TIM1_BKIN/TIM3_CH1/PA6); no longer U3.40 (PB4/SPI1_MISO/SYS_NJTRST/TIM3_CH1)
- net at R1.2, U3.10 (ADC1_IN0/ADC2_IN0/SYS_WKUP/TIM2_CH1/TIM2_ETR/USART2_CTS/PA0): now also U3.11 (ADC1_IN1/ADC2_IN1/TIM2_CH2/USART2_RTS/PA1)
- net at U3.17 (ADC1_IN7/ADC2_IN7/SPI1_MOSI/TIM1_CH1N/TIM3_CH2/PA7): now also R21.2
- net at U3.41 (PB5/I2C1_SMBA/SPI1_MOSI/TIM3_CH2): no longer R21.2
Other:
- moved on the sheet: R21, R4, R5
Changed lines of the file:
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@@
     (title "Volume fix for audi concert1/chorus1 made by Blaupunkt")
     (date "2018-09-21")
-    (rev "4.0")
+    (rev "5.0")
     (comment 1 "Standalone version")
     (comment 2 "Author: Tomas Kovacik")
   )
   (junction (at 62.23 100.33))
-  (junction (at 123.19 92.71))
   (junction (at 123.698 118.11))
   (junction (at 134.62 97.79))
@@
   (junction (at 212.09 35.56))
   (junction (at 212.09 135.89))
+  (junction (at 288.4424 82.55))
+  (junction (at 300.99 97.79))
   (junction (at 303.53 220.98))
   (junction (at 332.74 110.49))
@@
     (stroke (width 0) (type solid) (color 0 0 0 0))
   )
-  (wire (pts (xy 105.41 90.17) (xy 124.46 90.17))
-    (stroke (width 0) (type solid) (color 0 0 0 0))
-  )
-  (wire (pts (xy 105.41 92.71) (xy 123.19 92.71))
-    (stroke (width 0) (type solid) (color 0 0 0 0))
-  )
   (wire (pts (xy 107.95 87.63) (xy 124.46 87.63))
     (stroke (width 0) (type solid) (color 0 0 0 0))
@@
     (stroke (width 0) (type solid) (color 0 0 0 0))
   )
-  (wire (pts (xy 123.19 92.71) (xy 124.46 92.71))
-    (stroke (width 0) (type solid) (color 0 0 0 0))
-  )
-  (wire (pts (xy 123.19 95.25) (xy 123.19 92.71))
-    (stroke (width 0) (type solid) (color 0 0 0 0))
-  )
-  (wire (pts (xy 123.19 95.25) (xy 124.46 95.25))
-    (stroke (width 0) (type solid) (color 0 0 0 0))
-  )
   (wire (pts (xy 123.698 118.11) (xy 124.46 118.11))
     (stroke (width 0) (type solid) (color 0 0 0 0))
@@
     (stroke (width 0) (type solid) (color 0 0 0 0))
   )
-  (wire (pts (xy 132.08 92.71) (xy 138.43 92.71))
-    (stroke (width 0) (type solid) (color 0 0 0 0))
-  )
-  (wire (pts (xy 132.08 95.25) (xy 138.43 95.25))
-    (stroke (width 0) (type solid) (color 0 0 0 0))
-  )
   (wire (pts (xy 132.08 97.79) (xy 134.62 97.79))
     (stroke (width 0) (type solid) (color 0 0 0 0))
@@
     (stroke (width 0) (type solid) (color 0 0 0 0))
   )
-  (wire (pts (xy 138.43 90.17) (xy 132.08 90.17))
-    (stroke (width 0) (type solid) (color 0 0 0 0))
-  )
   (wire (pts (xy 138.43 113.03) (xy 116.332 113.03))
     (stroke (width 0) (type solid) (color 0 0 0 0))
@@
     (stroke (width 0) (type solid) (color 0 0 0 0))
   )
+  (wire (pts (xy 285.75 82.55) (xy 288.4424 82.55))
+    (stroke (width 0) (type solid) (color 0 0 0 0))
+  )
+  (wire (pts (xy 285.75 85.09) (xy 288.417 85.09))
+    (stroke (width 0) (type solid) (color 0 0 0 0))
+  )
   (wire (pts (xy 285.75 90.17) (xy 308.102 90.17))
     (stroke (width 0) (type solid) (color 0 0 0 0))
@@
     (stroke (width 0) (type solid) (color 0 0 0 0))
   )
-  (wire (pts (xy 285.75 102.87) (xy 307.848 102.87))
+  (wire (pts (xy 285.75 95.25) (xy 292.1 95.25))
+    (stroke (width 0) (type solid) (color 0 0 0 0))
+  )
+  (wire (pts (xy 285.75 102.87) (xy 323.469 102.87))
     (stroke (width 0) (type solid) (color 0 0 0 0))
   )
@@
     (stroke (width 0) (type solid) (color 0 0 0 0))
   )
+  (wire (pts (xy 288.417 85.09) (xy 288.4424 82.55))
+    (stroke (width 0) (type solid) (color 0 0 0 0))
+  )
+  (wire (pts (xy 288.4424 82.55) (xy 294.64 82.55))
+    (stroke (width 0) (type solid) (color 0 0 0 0))
+  )
   (wire (pts (xy 290.068 120.65) (xy 290.068 140.97))
     (stroke (width 0) (type solid) (color 0 0 0 0))
   )
-  (wire (pts (xy 294.64 82.55) (xy 285.75 82.55))
+  (wire (pts (xy 292.1 97.79) (xy 285.75 97.79))
+    (stroke (width 0) (type solid) (color 0 0 0 0))
+  )
+  (wire (pts (xy 292.1 100.33) (xy 285.75 100.33))
+    (stroke (width 0) (type solid) (color 0 0 0 0))
+  )
+  (wire (pts (xy 300.99 97.79) (xy 299.72 97.79))
+    (stroke (width 0) (type solid) (color 0 0 0 0))
+  )
+  (wire (pts (xy 300.99 100.33) (xy 299.72 100.33))
+    (stroke (width 0) (type solid) (color 0 0 0 0))
+  )
+  (wire (pts (xy 300.99 100.33) (xy 300.99 97.79))
     (stroke (width 0) (type solid) (color 0 0 0 0))
   )
@@
   )
   (wire (pts (xy 311.15 220.98) (xy 303.53 220.98))
+    (stroke (width 0) (type solid) (color 0 0 0 0))
+  )
+  (wire (pts (xy 318.77 95.25) (xy 299.72 95.25))
+    (stroke (width 0) (type solid) (color 0 0 0 0))
+  )
+  (wire (pts (xy 318.77 97.79) (xy 300.99 97.79))
     (stroke (width 0) (type solid) (color 0 0 0 0))
   )
@@
     (effects (font (size 1.27 1.27)) (justify left bottom))
   )
-  (label "CLOCK_FROM_MCU" (at 105.41 90.17 0)
-    (effects (font (size 1.27 1.27)) (justify left bottom))
-  )
-  (label "DATA_FROM_MCU" (at 105.41 92.71 0)
-    (effects (font (size 1.27 1.27)) (justify left bottom))
-  )
   (label "BOOT1" (at 107.95 87.63 0)
     (effects (font (size 1.27 1.27)) (justify left bottom))
@@
     (effects (font (size 1.27 1.27)) (justify right bottom))
   )
-  (label "#STATUS_TO_PANEL" (at 307.848 102.87 180)
-    (effects (font (size 1.27 1.27)) (justify right bottom))
-  )
   (label "#STATUS_FROM_MCU" (at 308.102 90.17 180)
     (effects (font (size 1.27 1.27)) (justify right bottom))
@@
   )
   (label "GALA" (at 309.88 82.55 180)
+    (effects (font (size 1.27 1.27)) (justify right bottom))
+  )
+  (label "CLOCK_FROM_MCU" (at 318.77 95.25 180)
+    (effects (font (size 1.27 1.27)) (justify right bottom))
+  )
+  (label "DATA_FROM_MCU" (at 318.77 97.79 180)
+    (effects (font (size 1.27 1.27)) (justify right bottom))
+  )
+  (label "#STATUS_TO_PANEL" (at 323.469 102.87 180)
     (effects (font (size 1.27 1.27)) (justify right bottom))
   )
@@
     )
   )
-  (symbol (lib_id "Device:R") (at 128.27 90.17 270) (unit 1)
-    (in_bom yes)
-    (property "Reference" "R4" (id 0) (at 128.27 90.17 90))
-    (property "Value" "1k" (id 1) (at 132.08 91.44 90))
-    (property "Footprint" "Resistors_SMD.pretty:R_0805_HandSoldering" (id 2) (at 128.27 88.392 90)
-      (effects (font (size 1.27 1.27)) hide)
-    )
-    (property "Datasheet" "~" (id 3) (at 128.27 90.17 0)
-      (effects (font (size 1.27 1.27)) hide)
-    )
-  )
-  (symbol (lib_id "Device:R") (at 128.27 92.71 90) (unit 1)
-    (in_bom yes)
-    (property "Reference" "R5" (id 0) (at 128.27 92.71 90))
-    (property "Value" "1k" (id 1) (at 132.08 93.98 90))
-    (property "Footprint" "Resistors_SMD.pretty:R_0805_HandSoldering" (id 2) (at 128.27 94.488 90)
-      (effects (font (size 1.27 1.27)) hide)
-    )
-    (property "Datasheet" "~" (id 3) (at 128.27 92.71 0)
-      (effects (font (size 1.27 1.27)) hide)
-    )
-  )
-  (symbol (lib_id "Device:R") (at 128.27 95.25 90) (unit 1)
-    (in_bom yes)
-    (property "Reference" "R21" (id 0) (at 128.27 95.25 90))
-    (property "Value" "10k" (id 1) (at 132.08 96.52 90))
-    (property "Footprint" "Resistors_SMD.pretty:R_0805_HandSoldering" (id 2) (at 128.27 97.028 90)
-      (effects (font (size 1.27 1.27)) hide)
-    )
-    (property "Datasheet" "~" (id 3) (at 128.27 95.25 0)
-      (effects (font (size 1.27 1.27)) hide)
-    )
-  )
   (symbol (lib_id "Device:R") (at 128.27 97.79 270) (unit 1)
     (in_bom yes)
@@
       (effects (font (size 1.27 1.27)) hide)
     )
+  )
+  (symbol (lib_id "Device:R") (at 295.91 95.25 90) (unit 1)
+    (in_bom yes)
+    (property "Reference" "R4" (id 0) (at 295.91 95.25 90))
+    (property "Value" "1k" (id 1) (at 292.1 93.98 90))
+    (property "Footprint" "Resistors_SMD.pretty:R_0805_HandSoldering" (id 2) (at 295.91 97.028 90)
+      (effects (font (size 1.27 1.27)) hide)
+    )
+    (property "Datasheet" "~" (id 3) (at 295.91 95.25 0)
+      (effects (font (size 1.27 1.27)) hide)
+    )
+  )
+  (symbol (lib_id "Device:R") (at 295.91 97.79 270) (mirror x) (unit 1)
+    (in_bom yes)
+    (property "Reference" "R5" (id 0) (at 295.91 97.79 90))
+    (property "Value" "1k" (id 1) (at 292.1 99.06 90))
+    (property "Footprint" "Resistors_SMD.pretty:R_0805_HandSoldering" (id 2) (at 295.91 99.568 90)
+      (effects (font (size 1.27 1.27)) hide)
+    )
+    (property "Datasheet" "~" (id 3) (at 295.91 97.79 0)
+      (effects (font (size 1.27 1.27)) hide)
+    )
+  )
+  (symbol (lib_id "Device:R") (at 295.91 100.33 270) (mirror x) (unit 1)
+    (in_bom yes)
+    (property "Reference" "R21" (id 0) (at 295.91 100.33 90))
+    (property "Value" "10k" (id 1) (at 292.1 101.6 90))
+    (property "Footprint" "Resistors_SMD.pretty:R_0805_HandSoldering" (id 2) (at 295.91 102.108 90)
+      (effects (font (size 1.27 1.27)) hide)
+    )
+    (property "Datasheet" "~" (id 3) (at 295.91 100.33 0)
+      (effects (font (size 1.27 1.27)) hide)
+    )

Commit message: HW v5
Parts:
- added R23: 1k, Resistors_SMD.pretty:R_0805_HandSoldering, symbol Device:R
- added R24: 100, Resistors_SMD.pretty:R_0805_HandSoldering, symbol Device:R
- R19: value 1k -> NP
Connections:
- net RESET: now also R24.1; no longer U4.2 (RESET)
- net RESET_KA: now also R23.1
- net at U3.40 (PB4/SPI1_MISO/SYS_NJTRST/TIM3_CH1): now also R1.2, U3.41 (PB5/I2C1_SMBA/SPI1_MOSI/TIM3_CH2)
- new net: R23.2, U3.10 (ADC1_IN0/ADC2_IN0/SYS_WKUP/TIM2_CH1/TIM2_ETR/USART2_CTS/PA0)
- new net: R24.2, U4.2 (RESET)
- now unconnected: U3.11 (ADC1_IN1/ADC2_IN1/TIM2_CH2/USART2_RTS/PA1)
Other:
- note added: "Using the first SPI port (SPI_1) SS <--> PA4 <--> BOARD_SPI1_NSS_PIN SCK <--> PA5 <--> BOARD_SPI1_SCK_PIN MISO <--> PA6 <--> BOARD_SPI1_MISO_PIN MOSI <--> PA7 <--> BOARD_SPI1_MOSI_PIN"
- note added: "Using the second SPI port (SPI_2) SS <--> PB12 <--> BOARD_SPI2_NSS_PIN SCK <--> PB13 <--> BOARD_SPI2_SCK_PIN MISO <--> PB14 <--> BOARD_SPI2_MISO_PIN MOSI <--> PB15 <--> BOARD_SPI2_MOSI_PIN"
- moved on the sheet: R1, U4

Commit message: V5
Parts:
- C2, C3: value 22p -> 12p(NP)
- R15, R16: value 1k -> 1k(NP)
- R19: value NP -> 1k(NP)
- R22: value 10k -> 10k(NP)
- R24: value 100 -> 1k(NP)
- U4: value MAX809 -> MAX809(NP)
- Y1: value 32.768kHz -> 32.768kHz(NP)
Other:
- note added: "//V5 version //RESET_KA = PA0 //GALA = PB4 //mcuCLK = PA5 //mcuDATA = PA6 //mcuSTATUS = PA15"
Changed lines of the file:
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@@
+    (effects (font (size 1.27 1.27)) (justify left bottom))
+  )
+  (text "//V5 version \n//RESET_KA = PA0\n//GALA = PB4\n//mcuCLK = PA5\n//mcuDATA = PA6\n//mcuSTATUS = PA15"
+    (at 38.2524 170.7896 0)
     (effects (font (size 1.27 1.27)) (justify left bottom))
   )
@@
     (in_bom yes)
     (property "Reference" "R19" (id 0) (at 128.27 102.87 90))
-    (property "Value" "NP" (id 1) (at 132.08 104.14 90))
+    (property "Value" "1k(NP)" (id 1) (at 132.08 104.14 90))
     (property "Footprint" "Resistors_SMD.pretty:R_0805_HandSoldering" (id 2) (at 128.27 104.648 90)
       (effects (font (size 1.27 1.27)) hide)
@@
     )
   )
-  (symbol (lib_id "Device:R") (at 128.27 115.57 90) (mirror x) (unit 1)
+  (symbol (lib_name "Device:R_1") (lib_id "Device:R") (at 128.27 115.57 90) (mirror x) (unit 1)
     (in_bom yes)
     (property "Reference" "R15" (id 0) (at 128.27 115.57 90))
-    (property "Value" "1k" (id 1) (at 132.08 116.84 90))
+    (property "Value" "1k(NP)" (id 1) (at 132.08 116.84 90))
     (property "Footprint" "Resistors_SMD.pretty:R_0805_HandSoldering" (id 2) (at 128.27 113.792 90)
       (effects (font (size 1.27 1.27)) hide)
@@
     )
   )
-  (symbol (lib_id "Device:R") (at 128.27 118.11 90) (mirror x) (unit 1)
+  (symbol (lib_name "Device:R_2") (lib_id "Device:R") (at 128.27 118.11 90) (mirror x) (unit 1)
     (in_bom yes)
     (property "Reference" "R16" (id 0) (at 128.27 118.11 90))
-    (property "Value" "1k" (id 1) (at 132.08 119.38 90))
+    (property "Value" "1k(NP)" (id 1) (at 132.08 119.38 90))
     (property "Footprint" "Resistors_SMD.pretty:R_0805_HandSoldering" (id 2) (at 128.27 116.332 90)
       (effects (font (size 1.27 1.27)) hide)
@@
     (in_bom yes)
     (property "Reference" "R22" (id 0) (at 128.27 120.65 90))
-    (property "Value" "10k" (id 1) (at 132.08 121.92 90))
+    (property "Value" "10k(NP)" (id 1) (at 132.08 121.92 90))
     (property "Footprint" "Resistors_SMD.pretty:R_0805_HandSoldering" (id 2) (at 128.27 122.428 90)
       (effects (font (size 1.27 1.27)) hide)
@@
     (in_bom yes)
     (property "Reference" "R24" (id 0) (at 344.17 38.1 90))
-    (property "Value" "100" (id 1) (at 343.9922 35.7378 90))
+    (property "Value" "1k(NP)" (id 1) (at 343.992 35.738 90))
     (property "Footprint" "Resistors_SMD.pretty:R_0805_HandSoldering" (id 2) (at 344.17 36.322 90)
       (effects (font (size 1.27 1.27)) hide)
@@
       (effects (font (size 1.27 1.27)) (justify left))
     )
-    (property "Value" "32.768kHz" (id 1) (at 371.8814 104.013 90)
+    (property "Value" "32.768kHz(NP)" (id 1) (at 371.881 104.013 90)
       (effects (font (size 1.27 1.27)) (justify left))
     )
@@
       (effects (font (size 1.524 1.524)))
     )
-    (property "Value" "22p" (id 1) (at 346.71 91.8972 90)
+    (property "Value" "12p(NP)" (id 1) (at 346.71 91.897 90)
       (effects (font (size 1.524 1.524)))
     )
@@
       (effects (font (size 1.524 1.524)))
     )
-    (property "Value" "22p" (id 1) (at 346.71 105.8672 90)
+    (property "Value" "12p(NP)" (id 1) (at 346.71 105.867 90)
       (effects (font (size 1.524 1.524)))
     )
@@
       (effects (font (size 1.27 1.27)) (justify right))
     )
-    (property "Value" "MAX809" (id 1) (at 314.2488 39.243 0)
+    (property "Value" "MAX809(NP)" (id 1) (at 314.249 39.243 0)
       (effects (font (size 1.27 1.27)) (justify right))
     )
