File: HW/audi_concert1_chorus1_volume_fix/audi_concert1_chorus1_volume_fix.kicad_sch (KiCad schematic)
At the start: 44 parts, among them CON1 I2C_to_TDA, CON2 USB, CON3 SPI_TO_PANEL, CON4 JLINK, U1 68HC05_PLCC, U2 AP1117-33, U3 STM32F103C8Tx, U4 MAX809(NP), Y1 32.768kHz(NP), Y2 8MHz

Commit message: hwv5
Parts:
- R12, R13: value 20 -> 20(NP)
- R14: value 1k5 -> 1k5(NP)
- R17: value 1k -> 1k(NP)
Changed lines of the file:
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@@
   )
   (text "    Using the second SPI port (SPI_2)\n    SS    <-->  PB12 <-->  BOARD_SPI2_NSS_PIN\n    SCK   <-->  PB13 <-->  BOARD_SPI2_SCK_PIN\n    MISO  <-->  PB14 <-->  BOARD_SPI2_MISO_PIN\n    MOSI  <-->  PB15 <-->  BOARD_SPI2_MOSI_PIN\n"
-    (at 127.2032 138.5062 0)
+    (at 127.2032 138.5062 180)
     (effects (font (size 1.27 1.27)) (justify right bottom))
   )
@@
   )
   (text "    Using the first SPI port (SPI_1)\n    SS    <-->  PA4 <-->  BOARD_SPI1_NSS_PIN\n    SCK   <-->  PA5 <-->  BOARD_SPI1_SCK_PIN\n    MISO  <-->  PA6 <-->  BOARD_SPI1_MISO_PIN\n    MOSI  <-->  PA7 <-->  BOARD_SPI1_MOSI_PIN"
-    (at 370.8908 84.6836 0)
+    (at 370.8908 84.6836 180)
     (effects (font (size 1.27 1.27)) (justify right bottom))
   )
@@
     (in_bom yes) (on_board yes)
     (property "Reference" "R12" (id 0) (at 54.61 100.33 90))
-    (property "Value" "20" (id 1) (at 58.42 101.6 90))
+    (property "Value" "20(NP)" (id 1) (at 58.42 101.6 90))
     (property "Footprint" "Resistors_SMD.pretty:R_0805_HandSoldering" (id 2) (at 54.61 98.552 90)
       (effects (font (size 1.27 1.27)) hide)
@@
     (in_bom yes) (on_board yes)
     (property "Reference" "R13" (id 0) (at 54.61 104.14 90))
-    (property "Value" "20" (id 1) (at 58.42 105.41 90))
+    (property "Value" "20(NP)" (id 1) (at 58.42 105.41 90))
     (property "Footprint" "Resistors_SMD.pretty:R_0805_HandSoldering" (id 2) (at 54.61 105.918 90)
       (effects (font (size 1.27 1.27)) hide)
@@
     (in_bom yes) (on_board yes)
     (property "Reference" "R14" (id 0) (at 62.23 92.71 90))
-    (property "Value" "1k5" (id 1) (at 63.5 87.63 90))
+    (property "Value" "1k5(NP)" (id 1) (at 63.5 87.63 90))
     (property "Footprint" "Resistors_SMD.pretty:R_0805_HandSoldering" (id 2) (at 64.008 92.71 90)
       (effects (font (size 1.27 1.27)) hide)
@@
     (in_bom yes) (on_board yes)
     (property "Reference" "R17" (id 0) (at 128.143 85.09 90))
-    (property "Value" "1k" (id 1) (at 131.953 86.36 90))
+    (property "Value" "1k(NP)" (id 1) (at 131.953 86.36 90))
     (property "Footprint" "Resistors_SMD.pretty:R_0805_HandSoldering" (id 2) (at 128.143 83.312 90)
       (effects (font (size 1.27 1.27)) hide)
@@
     )
     (path "/00000000-0000-0000-0000-00005ad5db61"
-      (reference "R12") (unit 1) (value "20") (footprint "Resistors_SMD.pretty:R_0805_HandSoldering")
+      (reference "R12") (unit 1) (value "20(NP)") (footprint "Resistors_SMD.pretty:R_0805_HandSoldering")
     )
     (path "/00000000-0000-0000-0000-00005ad5ddb2"
-      (reference "R13") (unit 1) (value "20") (footprint "Resistors_SMD.pretty:R_0805_HandSoldering")
+      (reference "R13") (unit 1) (value "20(NP)") (footprint "Resistors_SMD.pretty:R_0805_HandSoldering")
     )
     (path "/00000000-0000-0000-0000-00005ad67c4f"
-      (reference "R14") (unit 1) (value "1k5") (footprint "Resistors_SMD.pretty:R_0805_HandSoldering")
+      (reference "R14") (unit 1) (value "1k5(NP)") (footprint "Resistors_SMD.pretty:R_0805_HandSoldering")
     )
     (path "/00000000-0000-0000-0000-00005ae4cc42"
@@
     )
     (path "/00000000-0000-0000-0000-00005ae4cd58"
-      (reference "R17") (unit 1) (value "1k") (footprint "Resistors_SMD.pretty:R_0805_HandSoldering")
+      (reference "R17") (unit 1) (value "1k(NP)") (footprint "Resistors_SMD.pretty:R_0805_HandSoldering")
     )
     (path "/00000000-0000-0000-0000-00005ad78ebb"

Commit message: HW update
Parts:
- C8: value 10u/16V -> 10u/16V(NP)
- R2: value 1k -> 3k3
- renumbered CON2 to CON2(NP)
Other:
- note added: "3V3/3k3=1mA"
- note added: "I2C to sound procesor"
- note added: "USB header - not used"
- note added: "boot configuration no botloader no solder bridges here"
- note added: "main crystal"
- note added: "power + power led"
- note added: "programing/debug header stlink serial"
- note added: "reset - not used"
- note added: "slow crystal - not used"
- note added: "socket for motorola mcu, mirrored"
- moved on the sheet: C2, C3, C4, C5, CON1, CON2(NP), CON3, CON4, D1, JP1, JP2, R1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
