File: HW/audi_concert1_chorus1_volume_fix/audi_concert1_chorus1_volume_fix_v4_for_v1_code.kicad_pcb (KiCad board)
At the start: 2 copper layers, 35.1 x 27.2 mm, 42 parts, among them CON1 I2C_to_TDA, CON2 USB, CON3 SPI_TO_PANEL, CON4 JLINK, U1 68HC05_PLCC, U2 AP1117-33, U3 STM32F103C8Tx, U4 MAX809, Y1 NP_32.768kHz, Y2 8MHz

Commit message: hw changes
Parts:
- CON3: value SPI_TO_PANEL -> NP_SPI_TO_PANEL
- R17: value 1k -> NP_1k
- R2: value 1k -> 10k
- R3, R8: value 1K -> 10k
Changed lines of the file:
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@@
       (effects (font (size 0.6 0.6) (thickness 0.1)))
     )
-    (fp_text value "1k" (at -0.12828 0.04826) (layer "F.Fab")
+    (fp_text value "NP_1k" (at -0.12828 0.04826) (layer "F.Fab")
       (effects (font (size 1 1) (thickness 0.15)))
     )
@@
       (effects (font (size 0.8 0.8) (thickness 0.125)))
     )
-    (fp_text value "1k" (at 0.00508 0.0254 90) (layer "F.Fab")
+    (fp_text value "10k" (at 0.00508 0.0254 90) (layer "F.Fab")
       (effects (font (size 1 1) (thickness 0.15)))
     )
@@
       (effects (font (size 0.8 0.8) (thickness 0.125)))
     )
-    (fp_text value "1K" (at 0.01016 -0.0508 90) (layer "F.Fab")
+    (fp_text value "10k" (at 0.01016 -0.0508 90) (layer "F.Fab")
       (effects (font (size 1 1) (thickness 0.15)))
     )
@@
       (effects (font (size 0.8 0.8) (thickness 0.1)))
     )
-    (fp_text value "1K" (at 0.04318 0.06604 90) (layer "F.Fab")
+    (fp_text value "10k" (at 0.04318 0.06604 90) (layer "F.Fab")
       (effects (font (size 1 1) (thickness 0.15)))
     )
@@
       (effects (font (size 0.6 0.6) (thickness 0.1)))
     )
-    (fp_text value "SPI_TO_PANEL" (at 7.76732 1.72974 180) (layer "F.Fab")
-      (effects (font (size 1 1) (thickness 0.15)))
-    )
+    (fp_text value "NP_SPI_TO_PANEL" (at 7.76732 1.72974 180) (layer "F.Fab")
+      (effects (font (size 1 1) (thickness 0.15)))
+    )

Commit message: V5
Parts:
- R1: value 1k_GALA -> 1k
- R12, R13: value 20 -> NP_20
- R14: value 1k5 -> NP_1k5
- R19: value 1k -> NP_1k
- R20: value NP_1k -> 1k
- R3, R8: value 10k -> 100k
- U4: value MAX809 -> NP_MAX809
Changed lines of the file:
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@@
       (effects (font (size 0.8 0.8) (thickness 0.1)))
     )
-    (fp_text value "NP_1k" (at 0.14224 0.08382 90) (layer "F.Fab")
+    (fp_text value "1k" (at 0.14224 0.08382 90) (layer "F.Fab")
       (effects (font (size 1 1) (thickness 0.15)))
     )
@@
       (effects (font (size 1 1) (thickness 0.15)))
     )
-    (fp_text value "MAX809" (at -2.50952 0.0635 180) (layer "F.Fab")
+    (fp_text value "NP_MAX809" (at -2.50952 0.0635 180) (layer "F.Fab")
       (effects (font (size 1 1) (thickness 0.15)))
     )
@@
       (effects (font (size 0.8 0.8) (thickness 0.125)))
     )
-    (fp_text value "10k" (at 0.01016 -0.0508 90) (layer "F.Fab")
+    (fp_text value "100k" (at 0.01016 -0.0508 90) (layer "F.Fab")
       (effects (font (size 1 1) (thickness 0.15)))
     )
@@
       (effects (font (size 1 1) (thickness 0.15)))
     )
-    (fp_text value "20" (at 0.0546 0.19558) (layer "F.Fab")
+    (fp_text value "NP_20" (at 0.0546 0.19558) (layer "F.Fab")
       (effects (font (size 1 1) (thickness 0.15)))
     )
@@
       (effects (font (size 1 1) (thickness 0.15)))
     )
-    (fp_text value "20" (at -0.12446 0.00254 180) (layer "F.Fab")
+    (fp_text value "NP_20" (at -0.12446 0.00254 180) (layer "F.Fab")
       (effects (font (size 1 1) (thickness 0.15)))
     )
@@
       (effects (font (size 0.8 0.8) (thickness 0.15)))
     )
-    (fp_text value "1k" (at -0.05334 -0.01524 90) (layer "F.Fab")
+    (fp_text value "NP_1k" (at -0.05334 -0.01524 90) (layer "F.Fab")
       (effects (font (size 1 1) (thickness 0.15)))
     )
@@
       (effects (font (size 0.8 0.8) (thickness 0.1)))
     )
-    (fp_text value "10k" (at 0.04318 0.06604 90) (layer "F.Fab")
+    (fp_text value "100k" (at 0.04318 0.06604 90) (layer "F.Fab")
       (effects (font (size 1 1) (thickness 0.15)))
     )
@@
       (effects (font (size 1 1) (thickness 0.15)))
     )
-    (fp_text value "1k5" (at -0.07746 -0.05334 180) (layer "F.Fab")
+    (fp_text value "NP_1k5" (at -0.07746 -0.05334 180) (layer "F.Fab")
       (effects (font (size 1 1) (thickness 0.15)))
     )
@@
       (effects (font (size 1 1) (thickness 0.15)))
     )
-    (fp_text value "1k_GALA" (at 0.0254 -0.0254) (layer "F.Fab")
-      (effects (font (size 1 1) (thickness 0.15)))
-    )
+    (fp_text value "1k" (at 0.0254 -0.0254) (layer "F.Fab")
+      (effects (font (size 1 1) (thickness 0.15)))
+    )
