File: HW/audi_concert1_chorus1_volume_fix/audi_concert1_chorus1_volume_fix_v4_for_v1_code.kicad_sch (KiCad schematic)
At the start: 42 parts, among them CON1 I2C_to_TDA, CON2 USB, CON3 NP_SPI_TO_PANEL, CON4 JLINK, U1 68HC05_PLCC, U2 AP1117-33, U3 STM32F103C8Tx, U4 MAX809, Y1 NP_32.768kHz, Y2 8MHz

Commit message: hw changes
Parts:
- R2: value 1k -> 10k
- R3, R8: value 1K -> 10k
Changed lines of the file:
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@@
     (in_bom yes)
     (property "Reference" "R3" (id 0) (at 128.27 87.63 90))
-    (property "Value" "1K" (id 1) (at 132.08 88.9 90))
+    (property "Value" "10k" (id 1) (at 132.08 88.9 90))
     (property "Footprint" "Resistors_SMD.pretty:R_0805_HandSoldering" (id 2) (at 128.27 85.852 90)
       (effects (font (size 1.27 1.27)) hide)
@@
     (in_bom yes)
     (property "Reference" "R8" (id 0) (at 129.54 54.61 90))
-    (property "Value" "1K" (id 1) (at 134.62 55.88 90))
+    (property "Value" "10k" (id 1) (at 134.62 55.88 90))
     (property "Footprint" "Resistors_SMD.pretty:R_0805_HandSoldering" (id 2) (at 129.54 52.832 90)
       (effects (font (size 1.27 1.27)) hide)
@@
     )
   )
-  (symbol (lib_id "Device:R") (at 360.68 234.95 180) (unit 1)
+  (symbol (lib_name "Device:R_2") (lib_id "Device:R") (at 360.68 234.95 180) (unit 1)
     (in_bom yes)
     (property "Reference" "R2" (id 0) (at 363.22 231.14 90))
-    (property "Value" "1k" (id 1) (at 363.22 237.49 90))
+    (property "Value" "10k" (id 1) (at 363.22 237.49 90))
     (property "Footprint" "Resistors_SMD.pretty:R_0805_HandSoldering" (id 2) (at 362.458 234.95 90)
       (effects (font (size 1.27 1.27)) hide)

Commit message: V5
Parts:
- R1: value 1k_GALA -> 1k
- R12, R13: value 20 -> NP_20
- R14: value 1k5 -> NP_1k5
- R19: value 1k -> NP_1k
- R20: value NP_1k -> 1k
- R3, R8: value 10k -> 100k
- U4: value MAX809 -> NP_MAX809
Changed lines of the file:
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@@
     (in_bom yes)
     (property "Reference" "R12" (id 0) (at 54.61 100.33 90))
-    (property "Value" "20" (id 1) (at 58.42 101.6 90))
+    (property "Value" "NP_20" (id 1) (at 58.42 101.6 90))
     (property "Footprint" "Resistors_SMD.pretty:R_0805_HandSoldering" (id 2) (at 54.61 98.552 90)
       (effects (font (size 1.27 1.27)) hide)
@@
     (in_bom yes)
     (property "Reference" "R13" (id 0) (at 54.61 104.14 90))
-    (property "Value" "20" (id 1) (at 58.42 105.41 90))
+    (property "Value" "NP_20" (id 1) (at 58.42 105.41 90))
     (property "Footprint" "Resistors_SMD.pretty:R_0805_HandSoldering" (id 2) (at 54.61 105.918 90)
       (effects (font (size 1.27 1.27)) hide)
@@
     (in_bom yes)
     (property "Reference" "R14" (id 0) (at 62.23 92.71 90))
-    (property "Value" "1k5" (id 1) (at 63.5 87.63 90))
+    (property "Value" "NP_1k5" (id 1) (at 63.5 87.63 90))
     (property "Footprint" "Resistors_SMD.pretty:R_0805_HandSoldering" (id 2) (at 64.008 92.71 90)
       (effects (font (size 1.27 1.27)) hide)
@@
     (in_bom yes)
     (property "Reference" "R20" (id 0) (at 125.73 36.83 90))
-    (property "Value" "NP_1k" (id 1) (at 132.08 38.735 90))
+    (property "Value" "1k" (id 1) (at 132.08 38.735 90))
     (property "Footprint" "Resistors_SMD.pretty:R_0805_HandSoldering" (id 2) (at 125.73 38.608 90)
       (effects (font (size 1.27 1.27)) hide)
@@
     (in_bom yes)
     (property "Reference" "R3" (id 0) (at 128.27 87.63 90))
-    (property "Value" "10k" (id 1) (at 132.08 88.9 90))
+    (property "Value" "100k" (id 1) (at 132.08 88.9 90))
     (property "Footprint" "Resistors_SMD.pretty:R_0805_HandSoldering" (id 2) (at 128.27 85.852 90)
       (effects (font (size 1.27 1.27)) hide)
@@
     (in_bom yes)
     (property "Reference" "R19" (id 0) (at 128.27 102.87 90))
-    (property "Value" "1k" (id 1) (at 132.08 104.14 90))
+    (property "Value" "NP_1k" (id 1) (at 132.08 104.14 90))
     (property "Footprint" "Resistors_SMD.pretty:R_0805_HandSoldering" (id 2) (at 128.27 104.648 90)
       (effects (font (size 1.27 1.27)) hide)
@@
     (in_bom yes)
     (property "Reference" "R8" (id 0) (at 129.54 54.61 90))
-    (property "Value" "10k" (id 1) (at 134.62 55.88 90))
+    (property "Value" "100k" (id 1) (at 134.62 55.88 90))
     (property "Footprint" "Resistors_SMD.pretty:R_0805_HandSoldering" (id 2) (at 129.54 52.832 90)
       (effects (font (size 1.27 1.27)) hide)
@@
     (in_bom yes)
     (property "Reference" "R1" (id 0) (at 298.45 77.2922 90))
-    (property "Value" "1k_GALA" (id 1) (at 298.45 79.604 90))
+    (property "Value" "1k" (id 1) (at 298.45 79.604 90))
     (property "Footprint" "Resistors_SMD.pretty:R_0805_HandSoldering" (id 2) (at 298.45 80.772 90)
       (effects (font (size 1.27 1.27)) hide)
@@
       (effects (font (size 1.27 1.27)) (justify right))
     )
-    (property "Value" "MAX809" (id 1) (at 332.0288 39.243 0)
+    (property "Value" "NP_MAX809" (id 1) (at 332.029 39.243 0)
       (effects (font (size 1.27 1.27)) (justify right))
     )

Commit message: hwv5
Parts:
- C2, C3: value NP_22p -> (none); footprint Capacitors_SMD.pretty:C_0805_HandSoldering -> (none)
- C4, C5: value 22p -> (none); footprint Capacitors_SMD.pretty:C_0805_HandSoldering -> (none)
- C6, C7: value 100n -> (none); footprint Capacitors_SMD.pretty:C_0805_HandSoldering -> (none)
- C8: value 10u/16V -> (none); footprint Capacitors_Tantalum_SMD.pretty:TantalC_SizeA_EIA-3216_HandSoldering -> (none)
- CON1: value I2C_to_TDA -> (none); footprint Pin_Headers.pretty:Pin_Header_Straight_1x02 -> (none)
- CON2: value USB -> (none); footprint Pin_Headers.pretty:Pin_Header_Straight_1x04 -> (none)
- CON3: value NP_SPI_TO_PANEL -> (none); footprint Pin_Headers.pretty:Pin_Header_Straight_1x03 -> (none)
- CON4: value JLINK -> (none); footprint Pin_Headers.pretty:Pin_Header_Straight_1x06 -> (none)
- D1: value red -> (none); footprint LEDs.pretty:LED-1206 -> (none)
- JP1, JP2: value SolderJumper_3_Open -> (none); footprint Jumper:SolderJumper-3_P1.3mm_Open_RoundedPad1.0x1.5mm_NumberLabels -> (none)
- R1, R11, R20, R4, R5, R6, R7: value 1k -> (none); footprint Resistors_SMD.pretty:R_0805_HandSoldering -> (none)
- R10, R9: value 47k -> (none); footprint Resistors_SMD.pretty:R_0805_HandSoldering -> (none)
- R12, R13: value NP_20 -> (none); footprint Resistors_SMD.pretty:R_0805_HandSoldering -> (none)
- R14: value NP_1k5 -> (none); footprint Resistors_SMD.pretty:R_0805_HandSoldering -> (none)
- R15, R16, R17, R19: value NP_1k -> (none); footprint Resistors_SMD.pretty:R_0805_HandSoldering -> (none)
- R18: value 1M -> (none); footprint Resistors_SMD.pretty:R_0805_HandSoldering -> (none)
- R2: value 10k -> (none); footprint Resistors_SMD.pretty:R_0805_HandSoldering -> (none)
- R21, R22: value NP_10k -> (none); footprint Resistors_SMD.pretty:R_0805_HandSoldering -> (none)
- R3, R8: value 100k -> (none); footprint Resistors_SMD.pretty:R_0805_HandSoldering -> (none)
- U1: value 68HC05_PLCC -> (none); footprint modules:PLCC-52_mirrored -> (none)
- U2: value AP1117-33 -> (none); footprint ab2_sot.mod:AB2_SOT223 -> (none)
- U3: value STM32F103C8Tx -> (none); footprint Housings_QFP:LQFP-48_7x7mm_Pitch0.5mm -> (none)
- U4: value NP_MAX809 -> (none); footprint TO_SOT_Packages_SMD.pretty:SOT-23 -> (none)
- Y1: value NP_32.768kHz -> (none); footprint Crystals:Crystal_SMD_3215-2pin_3.2x1.5mm -> (none)
- Y2: value 8MHz -> (none); footprint Crystals:Crystal_SMD_5032-4pin_5.0x3.2mm -> (none)
